File: USBPD_Board.kicad_pcb (KiCad board)
At the start: 4 copper layers, 100 x 50 mm, 166 parts, among them IC1 STM32L100C6U6A, J10 Power_IO_JMP, J2 VSYS_Jmp, J3 USB_C_Receptacle_USB2.0_16P, J5 SWD1, J6 I2C1_Headers, J7 SWD2, J8 UART1_HDR, J9 ENABLE_JMP, M1 MOSFET_SI7155DP-T1-GE3, M2 MOSFET_SI7155DP-T1-GE3, M3 MOSFET_SI7155DP-T1-GE3, Q1 BSN20, Q2 BSN20, U4 MCP16331T-E/CH, U5 USBLC6-2SC6, U7 USBLC6-2SC6, U8 FSUSB42MUX

Commit message: Update
Parts:
- removed C1, C8: 1u 50V, Capacitor_SMD:C_0805_2012Metric
- removed C19, C31: 220p 50V NP0, Capacitor_SMD:C_0805_2012Metric
- removed C20, C5, C7: 100n 16V, Capacitor_SMD:C_0805_2012Metric
- removed C21, C22, C23, C24, C25, C26, C27, C28, C29, C46, C47, C48, C49: 100n, Capacitor_SMD:C_0805_2012Metric
- removed C4: 10u 16V, Capacitor_SMD:C_0805_2012Metric
- removed C9: 1u 100V X7T, Capacitor_SMD:C_0805_2012Metric
- removed D2: MMSZ5241BQ-7-F, Diode_SMD:D_SOD-123
- removed FB1: BLM21AG221SN1D 220 Ohms @ 100 MHz, Capacitor_SMD:C_0805_2012Metric
- removed J2: VSYS_Jmp, Connector_PinHeader_2.54mm:PinHeader_1x03_P2.54mm_Vertical
- removed J5: SWD1, Connector_PinHeader_2.54mm:PinHeader_2x04_P2.54mm_Horizontal
- removed J7: SWD2, Connector_PinHeader_2.54mm:PinHeader_2x04_P2.54mm_Horizontal
- removed J8: UART1_HDR, Connector_PinHeader_2.54mm:PinHeader_2x03_P2.54mm_Horizontal
- removed J9: ENABLE_JMP, Connector_PinHeader_2.54mm:PinHeader_1x03_P2.54mm_Vertical
- removed M2: MOSFET_SI7155DP-T1-GE3, Personal_Project:MOSFET_SI7155DPT1GE3
- removed Q1, Q2: BSN20, Package_TO_SOT_SMD:SOT-23
- removed R10, R61, R62, R63, R64, R9: 4k7, Resistor_SMD:R_0805_2012Metric
- removed R11: 100K, Resistor_SMD:R_0805_2012Metric
- removed R12, R13, R16, R5: 10K, Resistor_SMD:R_0805_2012Metric
- removed R14, R15, R17, R18, R19, R25, R50, R51, R52, R53: 100R, Resistor_SMD:R_0805_2012Metric
- removed R3: 226k, Resistor_SMD:R_0805_2012Metric
- removed R44: 33R, Resistor_SMD:R_0805_2012Metric
- removed R45, R54, R55, R56: 0.05R, Resistor_SMD:R_0805_2012Metric
- removed R46, R47, R48, R49, R57, R58, R59, R60: 0R, Resistor_SMD:R_0805_2012Metric
- removed R6: 300R, Resistor_SMD:R_1206_3216Metric
- removed U5, U7: USBLC6-2SC6, Package_TO_SOT_SMD:SOT-23-6
- removed U8: FSUSB42MUX, Package_SO:MSOP-10_3x3mm_P0.5mm
- removed UPD1: MCP22301T-2I/KYX, Personal_Project:USB_PD_MCP22301T_2I_KYX_VQFN40_KYX_MCH
- added D6: MMSZ5241BQ-7-F, Diode_SMD:D_SOD-123, B.Cu at (136.2, 83.8)
- added G***: LOGO, Personal_Project:PCB_Logo, B.Cu at (182.5, 86.2)
- added J1: I/O_HDR, Connector_PinHeader_2.54mm:PinHeader_2x04_P2.54mm_Horizontal, F.Cu at (125.0, 112.4)
- added S2: Switch_WS-SLSU SMT Mini Slide, Personal_Project:Switch_WS-SLSU SMT Mini Slide, B.Cu at (102.9, 95.1)
- added U2: USBLC6-2SC6, Package_TO_SOT_SMD:SOT-23-6, F.Cu at (112.9, 105.7)
- C10, C11, C12, C13, C14, C15, C16, C17, C18, D4, D5, DI4, FB2, L1, LDO1, R20, R21, R24, R26, U4, VS1: moved to B.Cu
- C3: value 100n 50V X7R -> 100n
- D1: value BAV99 -> SMA6S25AH; footprint Package_TO_SOT_SMD:SOT-23 -> Diode_SMD:D_SOD-123; moved to B.Cu
- IC1: value STM32L100C6U6A -> USB_MCP2221A-I_ST; footprint Personal_Project:QFN50P700X700X65-49N-D -> Personal_Project:SOP65P640X120-14N
- M1: moved to F.Cu
- R1: value 4k7 -> 100K; moved to B.Cu
- R2: value 4k7 -> 10K; moved to B.Cu
- R33, R35: value 5m_1% -> 5m_1%_CRE2512-FZ-R005E-2; footprint Resistor_SMD:R_0805_2012Metric -> Resistor_SMD:R_2512_6332Metric
- R4: value 10K -> 4k7
- R7: value 300R -> 5k1; footprint Resistor_SMD:R_1206_3216Metric -> Resistor_SMD:R_0805_2012Metric
- R8: value 10K -> 5k1
- moved FB2 203.9 mm to (115.6, 88.9)
- moved L1 200.8 mm to (116.3, 95.8), turned to 90 degrees
- moved D4 197.3 mm to (114.2, 100.0), turned to 180 degrees
- moved C10 194.7 mm to (115.5, 103.2), turned to 90 degrees
- moved C13 193.6 mm to (111.8, 88.9), turned to 180 degrees
- moved C12 192.4 mm to (111.8, 91.5), turned to 180 degrees
- moved R20 192.2 mm to (116.2, 91.5), turned to 0 degrees
- moved D5 191.0 mm to (120.7, 95.8), turned to 90 degrees
- moved C11 187.5 mm to (118.9, 100.0), turned to 180 degrees
- moved U4 187.4 mm to (118.9, 103.2), turned to 180 degrees
- moved C30 186.0 mm to (114.0, 114.8), turned to 90 degrees
- moved R21 182.7 mm to (120.6, 90.1), turned to 90 degrees
- moved U6 182.1 mm to (112.4, 118.7), turned to 90 degrees
- moved R27 177.2 mm to (113.2, 111.8), turned to 180 degrees
- moved IC1 139.0 mm to (123.5, 106.0), turned to 180 degrees
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Connections:
- net /USB/D+ renamed /USB/USB_D2+
- net /USB/D- renamed /USB/USB_D2-
- net Net-(D4-K) renamed /SMPS_LDO/MCP16331_SW
- net Net-(D5-A) renamed /SMPS_LDO/MCP16331_LOUT
- net Net-(D5-K) renamed /SMPS_LDO/MCP16331_BOOST
- net Net-(J10-Pin_1) renamed /Power_IO/CONN1+
- net Net-(J10-Pin_3) renamed /Power_IO/CONN2+
- net Net-(MS1-D_1) renamed /MCP19061/D_MS1
- net Net-(MS1-S_1) renamed /MCP19061/D_MS2
- net Net-(MS3-S_1) renamed /MCP19061/D_MS4
- net Net-(U4-V_{FB}) renamed /SMPS_LDO/MCP16331_V_{FB}
- C10 pad 1: VBUS -> +VIN_SMPS
- C3 pad 1: /USB_PD/VBUS_DET_IN -> +3.3V
- C30 pad 2: /Interfaces/NRST1 -> /Interfaces/RST_BTN
- C32 pad 1: +5V -> +VIN_SMPS
- C50 pad 1: +5V -> +3.3V
- D1 pad 1: GND -> /Power_IO/+VIN_S
- D1 pad 2: +3.3V -> GND
- IC1 pad 1: /MCU_STM32L100C6U6A/VLCD -> +3.3V
- IC1 pad 10: /MCP19061/NALERT -> /Interfaces/I2C1_SCL_HDR
- IC1 pad 11: /MCU_STM32L100C6U6A/PA1/ADC_IN1 -> +3.3V
- IC1 pad 12: /MCU_STM32L100C6U6A/PA2/USART2_TX -> /USB/USB_D1+
- IC1 pad 13: /MCU_STM32L100C6U6A/PA3/USART2_RX -> /USB/USB_D1-
- IC1 pad 14: /MCU_STM32L100C6U6A/PA4/ADC_IN4 -> GND
- IC1 pad 2: /MCU_STM32L100C6U6A/PC13-WKUP2 -> /Interfaces/I/O_HDR2
- IC1 pad 3: /MCU_STM32L100C6U6A/PC14-OSC32_IN -> /Interfaces/I/O_HDR3
- IC1 pad 4: /MCU_STM32L100C6U6A/PC15-OSC32_OUT -> /Interfaces/RST_BTN
- IC1 pad 5: /MCU_STM32L100C6U6A/PH0-OSC_IN -> unconnected-(IC1-URX-Pad5)
- IC1 pad 6: /MCU_STM32L100C6U6A/PH1-OSC_OUT -> unconnected-(IC1-UTX-Pad6)
- IC1 pad 7: /Interfaces/NRST1 -> /USB/GP2
- IC1 pad 8: GND -> /USB/GP3
- IC1 pad 9: +3.3VA -> /Interfaces/I2C1_SDA_HDR
- J10 pad 2: +VIN_SMPS -> /Power_IO/+VIN_S
- J10 pad 4: +VIN_SMPS -> /Power_IO/+VIN_S
- J10 pad 6: +VIN_SMPS -> /Power_IO/+VIN_S
- J10 pad 8: +VIN_SMPS -> /Power_IO/+VIN_S
- J3 pad A4: VBUS -> VBUS_PWR+
- J3 pad A9: VBUS -> VBUS_PWR+
- J3 pad B4: VBUS -> VBUS_PWR+
- J3 pad B9: VBUS -> VBUS_PWR+
- JST1 pad 3: /Interfaces/NRST1 -> /Interfaces/RST_BTN
- JST2 pad 3: /Interfaces/NRST1 -> /Interfaces/RST_BTN
- JST3 pad 3: /Interfaces/NRST1 -> /Interfaces/RST_BTN
- JST4 pad 3: /Interfaces/NRST1 -> /Interfaces/RST_BTN
- M1 pad 1: /USB_PD/VBUS_S -> /Power_IO/+VIN_S
- M1 pad 2: /USB_PD/VBUS_S -> /Power_IO/+VIN_S
- M1 pad 3: /USB_PD/VBUS_S -> /Power_IO/+VIN_S
- M1 pad 4: Net-(D2-A) -> /Power_IO/ONF_GATE
- M1 pad 5: VBUS -> +VIN_SMPS
- MS3 pad 5: Net-(MS3-D_1) -> /MCP19061/D_MS3
- R1 pad 1: /Interfaces/SWDIO2 -> /Power_IO/ONF_GATE
- R1 pad 2: +3.3V -> /Power_IO/+VIN_S
- R2 pad 1: /Interfaces/SWCLK2 -> /Power_IO/ONF_GATE
- R2 pad 2: +3.3V -> Net-(R2-Pad2)
- R27 pad 1: /Interfaces/NRST1 -> /Interfaces/RST_BTN
- R35 pad 1: +VOUT_SMPS -> /MCP19061/D_MS3
- R35 pad 2: Net-(MS3-D_1) -> +VOUT_SMPS
- R36 pad 1: Net-(MS3-D_1) -> /MCP19061/D_MS3
- R4 pad 1: GND -> +3.3V
- R4 pad 2: /USB_PD/VBUS_DET_IN -> /MCP19061/ENABLE
- R7 pad 1: VBUS -> /USB/CC2
- R7 pad 2: Net-(Q1-D) -> GND
- R8 pad 1: GND -> /USB/CC1
- R8 pad 2: /USB_PD/GPIO8/VBUS_DIS -> GND
- SMPS1 pad 1: /Interfaces/NRST1 -> /Interfaces/RST_BTN
- SMPS1 pad 14: +5V -> +VIN_SMPS
- SMPS1 pad 4: /MCP19061/SCL -> /Interfaces/I2C1_SCL_HDR
- SMPS1 pad 5: /MCP19061/SDA -> /Interfaces/I2C1_SDA_HDR
- SMPS1 pad 6: /MCP19061/NALERT -> /Interfaces/I/O_HDR0
- SMPS1 pad 7: /MCP19061/SYNC -> /Interfaces/I/O_HDR1
- SMPS1 pad 8: +5V -> +3.3V
- U4 pad 4: VBUS -> +VIN_SMPS
- U4 pad 5: VBUS -> +VIN_SMPS
- U6 pad 1: /Interfaces/NRST1 -> /Interfaces/RST_BTN
- U6 pad 2: /Interfaces/NRST1 -> /Interfaces/RST_BTN
- VS1 pad 1: /Interfaces/NRST1 -> /Interfaces/RST_BTN
Routing:
- net /Interfaces/RST_BTN: track 0.00 -> 209.2 mm, vias 0 -> 2
- net +3.3V: track 0.00 -> 162.1 mm, vias 0 -> 5
- net /Interfaces/I/O_HDR1: track 0.00 -> 154.6 mm, vias 0 -> 1
- net /Interfaces/I/O_HDR0: track 0.00 -> 146.7 mm, vias 0 -> 1
- net /Interfaces/I2C1_SCL_HDR: track 0.00 -> 122.4 mm, vias 0 -> 4
- net /Interfaces/I2C1_SDA_HDR: track 0.00 -> 121.7 mm, vias 0 -> 4
- net +5V: track 0.00 -> 91.9 mm, vias 0 -> 2
- net GND: track 0.00 -> 75.4 mm, vias 0 -> 119
- net Net-(R2-Pad2): track 0.00 -> 70.3 mm, vias 0 -> 2
- net +VIN_SMPS: track 0.00 -> 64.7 mm, vias 0 -> 2
- net /MCP19061/ISPIN: track 0.00 -> 48.7 mm, vias 0 -> 2
- net /MCP19061/ISNIN: track 0.00 -> 44.2 mm, vias 0 -> 2
- net /MCP19061/ISNOUT: track 0.00 -> 38.8 mm, vias 0 -> 2
- net /MCP19061/ISPOUT: track 0.00 -> 34.6 mm, vias 0 -> 2
- net /MCP19061/HG2: track 0.00 -> 32.5 mm, vias 0 -> 2
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- added copper zone on F.Cu, net +VIN_SMPS
- added copper zone on B.Cu, net +VOUT_SMPS
- added copper zone on F.Cu, net +VOUT_SMPS
- added copper zone on F.Cu, net /MCP19061/D_MS1
- added copper zone on F.Cu, net /MCP19061/D_MS2
- added copper zone on F.Cu, net /MCP19061/D_MS3
- added copper zone on F.Cu, net /MCP19061/D_MS4
- added copper zone on F.Cu, net /Power_IO/+VIN_S
- added copper zone on F.Cu, net /Power_IO/CONN1+
- added copper zone on F.Cu, net /Power_IO/CONN2+
- added copper zone on F.Cu, net /Power_IO/MOSFET_PWR
- added copper zone on F.Cu, net /Power_IO/PWR+
- added copper zone on F.Cu, net /Power_IO/PWR+_PP
- added copper zone on B.Cu, net /SMPS_LDO/MCP16331_LOUT
- added copper zone on B.Cu, net /SMPS_LDO/MCP16331_SW
- added copper zone on F.Cu, net VBUS_PWR+
Other:
- board text added: "2.1"
- board text added: "2.5"
- board text added: "BAT"
- board text added: "CONN1"
- board text added: "CONN2"
- board text added: "I2C"
- board text added: "USB"

Commit message: Update
Parts:
- moved G*** 14.2 mm to (182.8, 100.4)
Connections:
- J1 pad 1: GND -> +3.3V
Routing:
- net +3.3V: track 162.1 -> 165.3 mm
- net GND: track 75.4 -> 73.0 mm, vias 119 -> 130
- net (no net): vias 0 -> 1
Other:
- board text added: "3V3"
- board text added: "GND"
- board text added: "RST"
- board text added: "USB-PD Board Revision: REV B Designer: Peter Hancak SMPS: MCP19061-E_RTB VIN: 35V (MAX)"
- board text added: "VOUT"

Commit message: Update
Parts:
- moved G*** 7.24 mm to (180.6, 107.3)
- moved R24 0.70 mm to (175.8, 92.5)
- moved R26 0.60 mm to (175.8, 94.7)
- moved R4 0.51 mm to (175.5, 95.2)
- moved R65 0.50 mm to (175.5, 93.0)
Routing:
- net GND: track 73.0 -> 99.4 mm, vias 130 -> 165
- net /Interfaces/I/O_HDR0: track 146.7 -> 148.8 mm
- net /Interfaces/I2C1_SCL_HDR: track 122.4 -> 120.5 mm
- net +3.3V: track 165.3 -> 166.8 mm
- net /Interfaces/I/O_HDR1: track 154.6 -> 156.0 mm
- net +VIN_SMPS: track 64.7 -> 65.8 mm
- net /Interfaces/I2C1_SDA_HDR: track 121.7 -> 121.1 mm
- net (no net): vias 1 -> 0
Other:
- board text added: "GP0"
- board text added: "GP1"
- board text added: "MCP19061"
- board text added: "MCP2221A"
- board text added: "NALERT"
- board text added: "SYNC"
- board text added: "USB TO I2C"
- board text added: "USB-PD Board Revision: REV B Designer: Peter Hancak SMPS: MCP19061-E_RTB I2C: 0x53 (10k on ADR0) USB TO I2C: MCP2221A VIN: 35V (MAX)"
- board text removed: "USB-PD Board Revision: REV B Designer: Peter Hancak SMPS: MCP19061-E_RTB VIN: 35V (MAX)"

Commit message: Update
Parts:
- added C1: 100n, Capacitor_SMD:C_0805_2012Metric, F.Cu at (139.0, 92.3)
- R1: value 100K -> 10K
- R65: value 4k7 -> 10k
Routing:
- net /Power_IO/ONF_GATE: track 20.5 -> 27.3 mm
- net GND: track 99.4 -> 105.4 mm, vias 165 -> 162
- net +3.3V: track 166.8 -> 167.3 mm
- net +5V: track 92.1 -> 91.6 mm

Commit message: Update
Parts:
- added G***: LOGO, Personal_Project:Logo_Polarity, B.Cu at (117.9, 72.5)
- added G***: LOGO, Personal_Project:Logo_Polarity, B.Cu at (130.2, 72.5)
- moved G*** 21.6 mm to (182.6, 85.8)
- moved R65 0.40 mm to (175.5, 92.6)
Other:
- board text added: "2.1 mm"
- board text added: "2.5 mm"
- board text added: "ADR0 I2CADDR"
- board text added: "I2C1"
- board text added: "MCP19061-E_RTB I2C ADDRESS 0x53 (10k on ADR0) R ON ADR0 I2C ADDR 1K 0x50 4K 0x51 6K 0x52 10K 0x53 11K 0x54 14K 0x55 16K 0x56 19K 0x57"
- board text added: "SCL"
- board text added: "SDA"
- board text added: "USB-PD Board Revision: REV B Designer: Peter Hancak SMPS: MCP19061-E_RTB USB TO I2C: MCP2221A VIN: 35V (MAX)"
- board text removed: "I2C"
- board text removed: "USB-PD Board Revision: REV B Designer: Peter Hancak SMPS: MCP19061-E_RTB I2C: 0x53 (10k on ADR0) USB TO I2C: MCP2221A VIN: 35V (MAX)"
