File: USB.kicad_sch (KiCad schematic)
At the start: 8 parts, among them J3 USB_C_Receptacle_USB2.0_16P, U2 USBLC6-2SC6

Commit message: Update
Parts:
- removed R10: 6k2, Resistor_SMD:R_0805_2012Metric, symbol Device:R
- removed R9: 10k, Resistor_SMD:R_0805_2012Metric, symbol Device:R
- added C3: 100n, Capacitor_SMD:C_0805_2012Metric, symbol Device:C
- added IC1: USB_MCP2221A-I_ST, Personal_Project:SOP65P640X120-14N, symbol Personal_Projects:USB_MCP2221A-I_ST
Connections:
- net GND: now also U2.2 (GND), C3.2, IC1.14 (VSS)
- net USB_D2+: now also U2.4 (I/O2); no longer U2.6 (I/O1)
- net USB_D2-: now also U2.6 (I/O1); no longer U2.4 (I/O2)
- net FSUSB42MUX_D+ renamed USB_D1+
- net USB_D1+: now also IC1.12 (D-)
- net FSUSB42MUX_D- renamed USB_D1-
- net USB_D1-: now also IC1.13 (D+)
- net VBUS renamed VBUS_PWR+
- new net +3.3V: C3.1, IC1.1 (VDD), IC1.11 (VUSB)
- new net GP0: IC1.2 (GP0)
- new net GP1: IC1.3 (GP1)
- new net GP2: IC1.7 (GP2)
- new net GP3: IC1.8 (GP3)
- new net SCL: IC1.10 (SCL)
- new net SDA: IC1.9 (SDA)
- new net ~{RST}: IC1.4 (~{RST})
- no-connect marks 2 -> 5
Other:
- moved on the sheet: C54, J3, R39, R7, R8, U2

Commit message: Update
Other:
- company: (none) -> Peter Hancak
- title: (none) -> USB-PD Board
Changed lines of the file:
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@@
 	(generator_version "8.0")
 	(paper "USLetter")
+	(title_block
+		(title "USB-PD Board")
+		(date "2025-12-03")
+		(rev "B")
+		(company "Peter Hancak")
+	)
 	(junction
 		(at 85.09 60.96)

Commit message: Update
Other:
- note added: "5V (3A MAX)"
- note removed: "3A - 5, 9, 15V 5A - 20, 28, 36, 48V"
Changed lines of the file:
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@@
 		)
 	)
-	(text "3A - 5, 9, 15V\n5A - 20, 28, 36, 48V"
+	(text "5V (3A MAX) "
 		(exclude_from_sim no)
-		(at 205.232 58.928 0)
+		(at 211.836 57.912 0)
 		(effects
 			(font
